File: module.kicad_sch (KiCad schematic)
At the start: 0 parts

Commit message: schematic completed
Parts:
- added AE401: Antenna_Shield, symbol Device:Antenna_Shield
- added C35, C36, C47: NC, Capacitor_SMD:C_0603_1608Metric_Pad1.08x0.95mm_HandSolder, symbol Device:C_Small
- added D401: LED2, LED_SMD:LED_0603_1608Metric_Pad1.05x0.95mm_HandSolder, symbol Device:LED_Small
- added D402: LED1, LED_SMD:LED_0603_1608Metric_Pad1.05x0.95mm_HandSolder, symbol Device:LED_Small
- added J2: USB_B_Micro, KH-MICRO5P-JN:KH-MICRO5P-JN, symbol Connector:USB_B_Micro
- added J401: UPDATE, Connector_PinSocket_2.54mm:PinSocket_1x05_P2.54mm_Vertical, symbol Connector_Generic:Conn_01x05
- added J404: PIO, Connector_PinSocket_2.54mm:PinSocket_1x08_P2.54mm_Vertical, symbol Connector_Generic:Conn_01x08
- added J405: NFC, Connector_PinSocket_2.54mm:PinSocket_1x02_P2.54mm_Vertical, symbol Connector_Generic:Conn_01x02
- added J406: UART, Connector_PinSocket_2.54mm:PinSocket_1x06_P2.54mm_Vertical, symbol Connector_Generic:Conn_01x06
- added J407: I2C, Connector_PinSocket_2.54mm:PinSocket_1x04_P2.54mm_Vertical, symbol Connector_Generic:Conn_01x04
- added JP401: LED1_S, Jumper:SolderJumper-2_P1.3mm_Bridged2Bar_RoundedPad1.0x1.5mm, symbol Jumper:Jumper_2_Small_Bridged
- added JP403: LED2_S, Jumper:SolderJumper-2_P1.3mm_Bridged2Bar_RoundedPad1.0x1.5mm, symbol Jumper:Jumper_2_Small_Bridged
- added R14: 0R, Resistor_SMD:R_0603_1608Metric_Pad0.98x0.95mm_HandSolder, symbol Device:R_Small
- added R15, R2: 22R, Resistor_SMD:R_0603_1608Metric_Pad0.98x0.95mm_HandSolder, symbol Device:R_Small
- added R31, R32: 1K, Resistor_SMD:R_0603_1608Metric_Pad0.98x0.95mm_HandSolder, symbol Device:R_Small
- added U401: ~, FSC-BT631D:FSC-BT631D, symbol FSC-BT631D:FSC-BT631D
Connections:
- new net: JP403.1 (A), R31.2
- new net: D402.2 (A), R32.1
- new net: JP401.1 (A), R32.2
- new net: C35.1, C36.2, U401.35 (RF)
- new net: AE401.1 (A), C35.2, C47.2
- new net: D401.2 (A), R31.1
- new net: R14.2, U401.9 (NC)
- new net +5V: J2.1 (VBUS)
- new net GND: AE401.2 (Shield), C36.1, C47.1, D401.1 (K), D402.1 (K), J2.5 (GND), J2.6 (Shield), J401.5 (Pin_5), J406.6 (Pin_6), J407.4 (Pin_4), U401.20 (GND), U401.25 (GND), U401.34 (GND), U401.36 (GND)
- new net MOD_D+: J2.3 (D+), R2.1
- new net MOD_D-: J2.2 (D-), R15.1
- new net P0.02/NFC1: J405.2 (Pin_2), U401.13 (P0.02/NFC1)
- new net P0.03/NFC2: J405.1 (Pin_1), U401.12 (P0.03/NFC2)
- new net P0.06: J404.7 (Pin_7), U401.7 (P0.06)
- new net P0.07: J404.6 (Pin_6), U401.6 (P0.07)
- new net P0.13/I2S_DIN: U401.16 (P0.13/I2S_IN)
- new net P0.14/I2S_BCLK: U401.15 (P0.14/I2S_CLK)
- new net P0.15/I2S_DOUT: U401.14 (P0.15/I2S_OUT)
- new net P0.16/I2S_WS: U401.17 (P0.16/I2S_SYNC)
- new net P0.22: J404.8 (Pin_8), U401.8 (P0.22)
- new net P0.23: J404.5 (Pin_5), U401.5 (P0.23)
- new net P0.24: J404.4 (Pin_4), U401.4 (P0.24)
- new net P0.25: J404.3 (Pin_3), U401.3 (P0.25)
- new net P0.26: J404.2 (Pin_2), U401.2 (P0.26)
- new net P0.27: J404.1 (Pin_1), U401.1 (P0.27)
- new net P1.00: JP403.2 (B), U401.22 (P1.00)
- new net P1.01: JP401.2 (B), U401.21 (P1.01)
- new net P1.02/I2C_SDA: J407.2 (Pin_2), U401.10 (P1.02/SDA)
- new net P1.03/I2C_SCL: J407.3 (Pin_3), U401.11 (P0.03/SCL)
- new net P1.08/UART_RXD: J406.3 (Pin_3), U401.32 (P1.08/UART_RXD)
- new net P1.09/UART_TXD: J406.4 (Pin_4), U401.31 (P1.09/UART_TXD)
- new net P1.10/UART_CTS: J406.2 (Pin_2), U401.33 (P1.10/UART_CTS_N)
- new net P1.1/UART_RTS: J406.5 (Pin_5), U401.30 (P1.11/UART_RTS)
- new net RESET: J401.4 (Pin_4), U401.23 (RESET)
- new net SWDCLK: J401.3 (Pin_3), U401.28 (SDWCLK)
- new net SWDIO: J401.2 (Pin_2), U401.29 (SWDIO)
- new net USB_D+: R2.2, U401.26 (USB_D+)
- new net USB_D-: R15.2, U401.27 (USB_D-)
- new net VBUS: U401.24 (VBUS)
- new net VDD: J401.1 (Pin_1), J406.1 (Pin_1), J407.1 (Pin_1), R14.1, U401.19 (VDD)
- no-connect marks 0 -> 2

Commit message: FINALISED LAYOUT
Parts:
- renumbered C35 to C401, C36 to C402, C47 to C403, D402 to D401, D401 to D402, J2 to J401, J401 to J402, J406 to J403, J407 to J404, J404 to J406, JP403 to JP402, R2 to R401, R15 to R402, R14 to R403, R32 to R404, R31 to R405
Connections:
- net VBUS is gone; now on net +5V: U401.24 (VBUS)

Commit message: finalised layout
Parts:
- renumbered AE401 to AE1, C401 to C20, C402 to C21, C403 to C22, D401 to D3, D402 to D4, J406 to J10, J401 to J5, J402 to J6, J403 to J7, J404 to J8, J405 to J9, JP401 to JP8, JP402 to JP9, R401 to R24, R402 to R25, R403 to R26, R404 to R27, R405 to R28, U401 to U3

Commit message: added ibom & fabrication files
Parts:
- AE1: footprint (none) -> Connector_Coaxial:U.FL_Hirose_U.FL-R-SMT-1_Vertical; now not fitted
Changed lines of the file:
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@@
 		(in_bom yes)
 		(on_board yes)
-		(dnp no)
+		(dnp yes)
 		(fields_autoplaced yes)
 		(property "Reference" "AE1"
@@
 			)
 		)
-		(property "Footprint" ""
+		(property "Footprint" "Connector_Coaxial:U.FL_Hirose_U.FL-R-SMT-1_Vertical"
 			(at 152.4 57.15 0)
 			(effects
