File: FSC-BT631D-Breakout.kicad_pcb (KiCad board)
At the start: 2 copper layers, 70.6 x 72.9 mm, 94 parts, among them IC1 TLV320AIC3204IRHBR, J1 USB_C_Receptacle_USB2.0_16P, J10 PIO, J2 M_EN, J3 LINE IN, J4 LINE OUT, J5 USB_B_Micro, J6 UPDATE, J7 UART, J8 I2C, J9 NFC, Q1 AONR21307, U1 HUSB238_002DD, U2 AP63203WU-7

Commit message: initial routing
Parts:
- added C23: 100pF, Capacitor_SMD:C_0603_1608Metric_Pad1.08x0.95mm_HandSolder, F.Cu at (167.6, 118.1)
- added C24: 100pF, Capacitor_SMD:C_0603_1608Metric_Pad1.08x0.95mm_HandSolder, F.Cu at (167.6, 120.7)
- added C25: 47uF, Capacitor_SMD:C_0603_1608Metric_Pad1.08x0.95mm_HandSolder, F.Cu at (180.3, 121.7)
- added C26: 47uF, Capacitor_SMD:C_0603_1608Metric_Pad1.08x0.95mm_HandSolder, F.Cu at (182.9, 121.9)
- added C27: 100nF, Capacitor_SMD:C_0603_1608Metric_Pad1.08x0.95mm_HandSolder, F.Cu at (198.1, 81.3)
- added C28: 100nF, Capacitor_SMD:C_0603_1608Metric_Pad1.08x0.95mm_HandSolder, F.Cu at (174.6, 106.0)
- added C29: 10uF, Capacitor_SMD:C_0603_1608Metric_Pad1.08x0.95mm_HandSolder, F.Cu at (174.6, 109.2)
- added C30: 100nF, Capacitor_SMD:C_0603_1608Metric_Pad1.08x0.95mm_HandSolder, F.Cu at (174.6, 93.6)
- added C31: 47uF, Capacitor_SMD:C_0603_1608Metric_Pad1.08x0.95mm_HandSolder, F.Cu at (174.6, 96.8)
- added C32: 100nF, Capacitor_SMD:C_0603_1608Metric_Pad1.08x0.95mm_HandSolder, F.Cu at (174.6, 99.7)
- added C33: 10uF, Capacitor_SMD:C_0603_1608Metric_Pad1.08x0.95mm_HandSolder, F.Cu at (174.6, 102.9)
- added C34: 3.3nF, Capacitor_SMD:C_0603_1608Metric_Pad1.08x0.95mm_HandSolder, F.Cu at (170.7, 93.6)
- added C35: 47nF, Capacitor_SMD:C_0603_1608Metric_Pad1.08x0.95mm_HandSolder, F.Cu at (170.7, 90.4)
- added C36: 22pF, Capacitor_SMD:C_0603_1608Metric_Pad1.08x0.95mm_HandSolder, F.Cu at (176.5, 85.7)
- added C37: 22pF, Capacitor_SMD:C_0603_1608Metric_Pad1.08x0.95mm_HandSolder, F.Cu at (186.7, 85.7)
- added C38: 5.6nF, Capacitor_SMD:C_0603_1608Metric_Pad1.08x0.95mm_HandSolder, F.Cu at (198.1, 66.0)
- added C39: 47uF, Capacitor_SMD:C_0603_1608Metric_Pad1.08x0.95mm_HandSolder, F.Cu at (198.1, 72.4)
- added C40: 47uF, Capacitor_SMD:C_0603_1608Metric_Pad1.08x0.95mm_HandSolder, F.Cu at (188.0, 73.0)
- added C41: 5.6nF, Capacitor_SMD:C_0603_1608Metric_Pad1.08x0.95mm_HandSolder, F.Cu at (188.0, 66.7)
- added C42: 47uF, Capacitor_SMD:C_0603_1608Metric_Pad1.08x0.95mm_HandSolder, F.Cu at (182.9, 73.0)
- added C43: 47uF, Capacitor_SMD:C_0603_1608Metric_Pad1.08x0.95mm_HandSolder, F.Cu at (172.7, 73.0)
- added C44: 5.6nF, Capacitor_SMD:C_0603_1608Metric_Pad1.08x0.95mm_HandSolder, F.Cu at (182.9, 66.7)
- added C45: 5.6nF, Capacitor_SMD:C_0603_1608Metric_Pad1.08x0.95mm_HandSolder, F.Cu at (172.7, 66.7)
- added C46: 100nF, Capacitor_SMD:C_0603_1608Metric_Pad1.08x0.95mm_HandSolder, F.Cu at (187.3, 122.6)
- added C47: 100nF, Capacitor_SMD:C_0603_1608Metric_Pad1.08x0.95mm_HandSolder, F.Cu at (191.1, 108.0)
- added C48: 100nF, Capacitor_SMD:C_0603_1608Metric_Pad1.08x0.95mm_HandSolder, F.Cu at (191.1, 100.3)
- added C49: 100uF, Capacitor_SMD:C_0603_1608Metric_Pad1.08x0.95mm_HandSolder, F.Cu at (194.9, 100.3)
- added C50: 100nF, Capacitor_SMD:C_0603_1608Metric_Pad1.08x0.95mm_HandSolder, F.Cu at (180.3, 93.3)
- added C51: 100nF, Capacitor_SMD:C_0603_1608Metric_Pad1.08x0.95mm_HandSolder, F.Cu at (182.9, 93.3)
- added C52: 100nF, Capacitor_SMD:C_0603_1608Metric_Pad1.08x0.95mm_HandSolder, F.Cu at (185.4, 93.3)
- added C53: 10uF, Capacitor_SMD:C_0603_1608Metric_Pad1.08x0.95mm_HandSolder, F.Cu at (177.8, 93.3)
- added C54: 10uF, Capacitor_SMD:C_0603_1608Metric_Pad1.08x0.95mm_HandSolder, F.Cu at (191.1, 94.0)
- added C55: 100nF, Capacitor_SMD:C_0603_1608Metric_Pad1.08x0.95mm_HandSolder, F.Cu at (191.1, 97.2)
- added J11: DSP IN, XKB_PJ-3200:XKB_PJ-3200, F.Cu at (177.7, 126.6)
- added J12: DSP_EN, Connector_PinSocket_2.54mm:PinSocket_1x02_P2.54mm_Vertical, F.Cu at (193.7, 125.1)
- added J13: OUT1, XKB_PJ-3200:XKB_PJ-3200, F.Cu at (190.6, 61.7)
- added J14: OUT2, XKB_PJ-3200:XKB_PJ-3200, F.Cu at (175.5, 61.9)
- added J15: SELFBOOT, Connector_PinHeader_2.54mm:PinHeader_1x03_P2.54mm_Vertical, F.Cu at (201.3, 116.2)
- added J16: DSP_PROG, Connector_PinSocket_2.54mm:PinSocket_1x05_P2.54mm_Vertical, F.Cu at (201.3, 106.0)
- added J17: DSP_GPIO, Connector_PinHeader_2.54mm:PinHeader_2x07_P2.54mm_Vertical, F.Cu at (167.0, 108.0)
- added Q2: BC807, Package_TO_SOT_SMD:SOT-23, F.Cu at (194.9, 104.1)
- added R30: 18K, Resistor_SMD:R_0603_1608Metric_Pad0.98x0.95mm_HandSolder, F.Cu at (180.3, 116.6)
- added R31: 18K, Resistor_SMD:R_0603_1608Metric_Pad0.98x0.95mm_HandSolder, F.Cu at (182.9, 116.8)
- added R32: 49.9k, Resistor_SMD:R_0603_1608Metric_Pad0.98x0.95mm_HandSolder, F.Cu at (167.6, 115.6)
- added R33: 49.9k, Resistor_SMD:R_0603_1608Metric_Pad0.98x0.95mm_HandSolder, F.Cu at (167.6, 123.2)
- added R34: 10k, Resistor_SMD:R_0603_1608Metric_Pad0.98x0.95mm_HandSolder, F.Cu at (191.8, 87.6)
- added R35: 10k, Resistor_SMD:R_0603_1608Metric_Pad0.98x0.95mm_HandSolder, F.Cu at (194.9, 87.6)
- added R36: 10k, Resistor_SMD:R_0603_1608Metric_Pad0.98x0.95mm_HandSolder, F.Cu at (198.1, 87.6)
- added R37: 18K, Resistor_SMD:R_0603_1608Metric_Pad0.98x0.95mm_HandSolder, F.Cu at (181.6, 110.5)
- added R38: 470R, Resistor_SMD:R_0603_1608Metric_Pad0.98x0.95mm_HandSolder, F.Cu at (170.7, 87.2)
- added R39: 100R, Resistor_SMD:R_0603_1608Metric_Pad0.98x0.95mm_HandSolder, F.Cu at (181.6, 90.2)
- added R40: 560R, Resistor_SMD:R_0603_1608Metric_Pad0.98x0.95mm_HandSolder, F.Cu at (198.1, 69.2)
- added R41: 560R, Resistor_SMD:R_0603_1608Metric_Pad0.98x0.95mm_HandSolder, F.Cu at (188.0, 69.8)
- added R42: 560R, Resistor_SMD:R_0603_1608Metric_Pad0.98x0.95mm_HandSolder, F.Cu at (182.9, 69.8)
- added R43: 560R, Resistor_SMD:R_0603_1608Metric_Pad0.98x0.95mm_HandSolder, F.Cu at (172.7, 69.8)
- added R44: 10K, Resistor_SMD:R_0603_1608Metric_Pad0.98x0.95mm_HandSolder, F.Cu at (187.3, 111.1)
- added R45: 1K, Resistor_SMD:R_0603_1608Metric_Pad0.98x0.95mm_HandSolder, F.Cu at (191.1, 104.1)
- added SW1: DSP_RST, TS3425BA:TS3425BA, F.Cu at (187.3, 116.8)
- added TP15: V_DSP, TestPoint:TestPoint_THTPad_1.0x1.0mm_Drill0.5mm, F.Cu at (196.2, 120.7)
- added TP16: 3.3V, TestPoint:TestPoint_THTPad_1.0x1.0mm_Drill0.5mm, F.Cu at (193.7, 120.7)
- added TP17: O1_R, TestPoint:TestPoint_THTPad_1.0x1.0mm_Drill0.5mm, F.Cu at (198.8, 62.9)
- added TP18: O1_L, TestPoint:TestPoint_THTPad_1.0x1.0mm_Drill0.5mm, F.Cu at (187.3, 62.9)
- added TP19: O2_R, TestPoint:TestPoint_THTPad_1.0x1.0mm_Drill0.5mm, F.Cu at (183.5, 62.9)
- added TP20: O2_L, TestPoint:TestPoint_THTPad_1.0x1.0mm_Drill0.5mm, F.Cu at (172.1, 62.9)
- added U4: ADAU1701, Package_QFP:LQFP-48_7x7mm_P0.5mm, F.Cu at (182.9, 101.6)
- added U5: M24C64-RMN6TP, Package_SO:SOIC-8_3.9x4.9mm_P1.27mm, F.Cu at (193.0, 81.3)
- added Y2: XTM32012288JT00351001, Crystal:Crystal_SMD_3225-4Pin_3.2x2.5mm_HandSoldering, F.Cu at (181.6, 85.7)
Connections:
- D4 pad 2: Net-(D4-A) -> unconnected-(R28-Pad1)
- JP8 pad 1: Net-(JP8-A) -> unconnected-(R27-Pad2)
- R26 pad 2: Net-(U3-NC) -> unconnected-(R26-Pad2)
- R27 pad 2: Net-(JP8-A) -> unconnected-(R27-Pad2)
- R28 pad 1: Net-(D4-A) -> unconnected-(R28-Pad1)
- U3 pad 18: unconnected-(U3-P0.12/I2S_MCLK-Pad18) -> (no net)
- U3 pad 9: Net-(U3-NC) -> unconnected-(R26-Pad2)
Routing:
- net unconnected-(R27-Pad2): track 0.00 -> 3.54 mm
- net Net-(JP8-A): track 3.54 -> 0.00 mm
- net unconnected-(R28-Pad1): track 0.00 -> 3.28 mm
- net Net-(D4-A): track 3.28 -> 0.00 mm
- net unconnected-(R26-Pad2): track 0.00 -> 2.80 mm
- net Net-(U3-NC): track 2.80 -> 0.00 mm
Other:
- board text added: "SBOOT"
- board text added: "VDSP"
- board text added: "WP"
