File: dsp.kicad_sch (KiCad schematic)
At the start: 67 parts, among them J11 DSP IN, J12 DSP_EN, J13 OUT1, J14 OUT2, J15 SELFBOOT, J16 DSP_PROG, J17 DSP_GPIO, Q2 BC807, SW1 DSP_RST, U4 ADAU1701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

Commit message: initial routing
Parts:
- TP16: value VDD -> 3.3V
Connections:
- net VDD renamed +3.3V
Changed lines of the file:
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@@
 	)
 	(junction
+		(at 190.5 64.77)
+		(diameter 0)
+		(color 0 0 0 0)
+	)
+	(junction
 		(at 96.52 129.54)
 		(diameter 0)
@@
 	(wire
 		(pts
+			(xy 195.58 60.96) (xy 195.58 64.77)
+		)
+		(stroke
+			(width 0)
+			(type default)
+		)
+	)
+	(wire
+		(pts
 			(xy 104.14 25.4) (xy 104.14 24.13)
 		)
@@
 	(wire
 		(pts
+			(xy 195.58 64.77) (xy 190.5 64.77)
+		)
+		(stroke
+			(width 0)
+			(type default)
+		)
+	)
+	(wire
+		(pts
 			(xy 129.54 30.48) (xy 129.54 31.75)
 		)
@@
 			)
 		)
-		(property "Value" "VDD"
+		(property "Value" "3.3V"
 			(at 170.434 68.326 90)
 			(effects
@@
 	)
 	(symbol
-		(lib_id "power:VDD")
-		(at 176.53 64.77 0)
+		(lib_id "power:GND")
+		(at 151.13 39.37 0)
 		(unit 1)
 		(exclude_from_sim no)
@@
 		(dnp no)
 		(fields_autoplaced yes)
-		(property "Reference" "#PWR055"
-			(at 176.53 68.58 0)
+		(property "Reference" "#PWR071"
+			(at 151.13 45.72 0)
 			(effects
 				(font
@@
 			)
 		)
-		(property "Value" "VDD"
-			(at 176.53 59.69 0)
+		(property "Value" "GND"
+			(at 151.13 44.45 0)
 			(effects
 				(font
@@
 		)
 		(property "Footprint" ""
-			(at 176.53 64.77 0)
+			(at 151.13 39.37 0)
 			(effects
 				(font
@@
 		)
 		(property "Datasheet" ""
-			(at 176.53 64.77 0)
+			(at 151.13 39.37 0)
 			(effects
 				(font
@@
 			)
 		)
-		(property "Description" "Power symbol creates a global label with name \"VDD\""
-			(at 176.53 64.77 0)
+		(property "Description" "Power symbol creates a global label with name \"GND\" , ground"
+			(at 151.13 39.37 0)
 			(effects
 				(font
@@
 		)
 		(instances
-			(project ""
+			(project "FSC-BT631D-Breakout"
 				(path "/484c4955-80b8-457c-864e-1c65a3218727/8996c219-c1ac-4183-83a9-3ce663da6e45"
-					(reference "#PWR055")
+					(reference "#PWR071")
 					(unit 1)
 				)
@@
 	)
 	(symbol
-		(lib_id "power:GND")
-		(at 151.13 39.37 0)
+		(lib_id "Device:C_Small")
+		(at 140.97 55.88 0)
 		(unit 1)
 		(exclude_from_sim no)
@@
 		(dnp no)
 		(fields_autoplaced yes)
-		(property "Reference" "#PWR071"
-			(at 151.13 45.72 0)
+		(property "Reference" "C37"
+			(at 143.51 54.6162 0)
 			(effects
 				(font
 					(size 1.27 1.27)
 				)
-				(hide yes)
+				(justify left)
 			)
 		)
-		(property "Value" "GND"
-			(at 151.13 44.45 0)
+		(property "Value" "22pF"
+			(at 143.51 57.1562 0)
 			(effects
 				(font
 					(size 1.27 1.27)
 				)
+				(justify left)
 			)
 		)
-		(property "Footprint" ""
-			(at 151.13 39.37 0)
+		(property "Footprint" "Capacitor_SMD:C_0603_1608Metric_Pad1.08x0.95mm_HandSolder"
+			(at 140.97 55.88 0)
 			(effects
 				(font
@@
 			)
 		)
-		(property "Datasheet" ""
-			(at 151.13 39.37 0)
+		(property "Datasheet" "~"
+			(at 140.97 55.88 0)
 			(effects
 				(font
@@
 			)
 		)
-		(property "Description" "Power symbol creates a global label with name \"GND\" , ground"
-			(at 151.13 39.37 0)
+		(property "Description" "Unpolarized capacitor, small symbol"
+			(at 140.97 55.88 0)
 			(effects
 				(font
@@
 			)
 		)
+		(pin "2"
+		)
 		(pin "1"
 		)
@@
 			(project "FSC-BT631D-Breakout"
 				(path "/484c4955-80b8-457c-864e-1c65a3218727/8996c219-c1ac-4183-83a9-3ce663da6e45"
-					(reference "#PWR071")
+					(reference "C37")
 					(unit 1)
 				)
@@
 	)
 	(symbol
-		(lib_id "Device:C_Small")
-		(at 140.97 55.88 0)
+		(lib_id "power:VDD")
+		(at 29.21 152.4 0)
 		(unit 1)
 		(exclude_from_sim no)
@@
 		(dnp no)
 		(fields_autoplaced yes)
-		(property "Reference" "C37"
-			(at 143.51 54.6162 0)
+		(property "Reference" "#PWR061"
+			(at 29.21 156.21 0)
 			(effects
 				(font
 					(size 1.27 1.27)
 				)
-				(justify left)
+				(hide yes)
 			)
 		)
-		(property "Value" "22pF"
-			(at 143.51 57.1562 0)
+		(property "Value" "V_DSP"
+			(at 29.21 147.32 0)
 			(effects
 				(font
 					(size 1.27 1.27)
 				)
-				(justify left)
 			)
 		)
-		(property "Footprint" "Capacitor_SMD:C_0603_1608Metric_Pad1.08x0.95mm_HandSolder"
-			(at 140.97 55.88 0)
+		(property "Footprint" ""
+			(at 29.21 152.4 0)
 			(effects
 				(font
@@
 			)
 		)
-		(property "Datasheet" "~"
-			(at 140.97 55.88 0)
+		(property "Datasheet" ""
+			(at 29.21 152.4 0)
 			(effects
 				(font
@@
 			)
 		)
-		(property "Description" "Unpolarized capacitor, small symbol"
-			(at 140.97 55.88 0)
+		(property "Description" "Power symbol creates a global label with name \"VDD\""
+			(at 29.21 152.4 0)
 			(effects
 				(font
@@
 			)
 		)
-		(pin "2"
-		)
 		(pin "1"
 		)
@@
 			(project "FSC-BT631D-Breakout"
 				(path "/484c4955-80b8-457c-864e-1c65a3218727/8996c219-c1ac-4183-83a9-3ce663da6e45"
-					(reference "C37")
+					(reference "#PWR061")
 					(unit 1)
 				)
@@
 	)
 	(symbol
-		(lib_id "power:VDD")
-		(at 29.21 152.4 0)
+		(lib_id "power:PWR_FLAG")
+		(at 195.58 60.96 0)
 		(unit 1)
 		(exclude_from_sim no)
@@
 		(dnp no)
 		(fields_autoplaced yes)
-		(property "Reference" "#PWR061"
-			(at 29.21 156.21 0)
+		(property "Reference" "#FLG05"
+			(at 195.58 59.055 0)
 			(effects
 				(font
@@
 			)
 		)
-		(property "Value" "V_DSP"
-			(at 29.21 147.32 0)
+		(property "Value" "PWR_FLAG"
+			(at 195.58 55.88 0)
 			(effects
 				(font
@@
 		)
 		(property "Footprint" ""
-			(at 29.21 152.4 0)
+			(at 195.58 60.96 0)
 			(effects
 				(font
@@
 			)
 		)
-		(property "Datasheet" ""
-			(at 29.21 152.4 0)
+		(property "Datasheet" "~"
+			(at 195.58 60.96 0)
 			(effects
 				(font
@@
 			)
 		)
-		(property "Description" "Power symbol creates a global label with name \"VDD\""
-			(at 29.21 152.4 0)
+		(property "Description" "Special symbol for telling ERC where power comes from"
+			(at 195.58 60.96 0)
 			(effects
 				(font
@@
 		)
 		(instances
-			(project "FSC-BT631D-Breakout"
+			(project ""
 				(path "/484c4955-80b8-457c-864e-1c65a3218727/8996c219-c1ac-4183-83a9-3ce663da6e45"
-					(reference "#PWR061")
+					(reference "#FLG05")
 					(unit 1)
 				)
@@
 					(unit 1)
 				)
+			)
+		)
+	)
+	(symbol
+		(lib_id "power:+3.3V")
+		(at 176.53 64.77 0)
+		(unit 1)
+		(exclude_from_sim no)
+		(in_bom yes)
+		(on_board yes)
+		(dnp no)
+		(fields_autoplaced yes)
+		(property "Reference" "#PWR084"
+			(at 176.53 68.58 0)
+			(effects
+				(font
+					(size 1.27 1.27)
+				)
+				(hide yes)
+			)
+		)
+		(property "Value" "+3.3V"
+			(at 176.53 59.69 0)
+			(effects
+				(font
+					(size 1.27 1.27)
+				)
+			)
+		)
+		(property "Footprint" ""
+			(at 176.53 64.77 0)
+			(effects
+				(font
+					(size 1.27 1.27)
+				)
+				(hide yes)
+			)
+		)
+		(property "Datasheet" ""
+			(at 176.53 64.77 0)
+			(effects
+				(font
+					(size 1.27 1.27)
+				)
+				(hide yes)
+			)
+		)
+		(property "Description" "Power symbol creates a global label with name \"+3.3V\""
+			(at 176.53 64.77 0)
+			(effects
+				(font
+					(size 1.27 1.27)
+				)
+				(hide yes)
+			)
+		)
+		(pin "1"
+		)
+		(instances
+			(project ""
+				(path "/484c4955-80b8-457c-864e-1c65a3218727/8996c219-c1ac-4183-83a9-3ce663da6e45"
+					(reference "#PWR084")
+					(unit 1)
+				)
