File: FSC-BT631D-Breakout/FSC-BT631D-Breakout.kicad_pcb (KiCad board)
At the start: 2 copper layers, 70.6 x 72.9 mm, 161 parts, among them IC1 TLV320AIC3204IRHBR, J1 USB_C_Receptacle_USB2.0_16P, J10 PIO, J11 DSP IN, J12 DSP_EN, J13 OUT1, J14 OUT2, J15 SELFBOOT, J16 DSP_PROG, J17 DSP_GPIO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

Commit message: folder restructure
Parts:
- removed C23, C24: 100pF, Capacitor_SMD:C_0603_1608Metric_Pad1.08x0.95mm_HandSolder
- removed C25, C26, C31, C39, C40, C42, C43: 47uF, Capacitor_SMD:C_0603_1608Metric_Pad1.08x0.95mm_HandSolder
- removed C27, C28, C30, C32, C46, C47, C48, C50, C51, C52, C55: 100nF, Capacitor_SMD:C_0603_1608Metric_Pad1.08x0.95mm_HandSolder
- removed C29, C33, C53, C54: 10uF, Capacitor_SMD:C_0603_1608Metric_Pad1.08x0.95mm_HandSolder
- removed C34: 3.3nF, Capacitor_SMD:C_0603_1608Metric_Pad1.08x0.95mm_HandSolder
- removed C35: 47nF, Capacitor_SMD:C_0603_1608Metric_Pad1.08x0.95mm_HandSolder
- removed C36, C37: 22pF, Capacitor_SMD:C_0603_1608Metric_Pad1.08x0.95mm_HandSolder
- removed C38, C41, C44, C45: 5.6nF, Capacitor_SMD:C_0603_1608Metric_Pad1.08x0.95mm_HandSolder
- removed C49: 100uF, Capacitor_SMD:C_0603_1608Metric_Pad1.08x0.95mm_HandSolder
- removed J11: DSP IN, XKB_PJ-3200:XKB_PJ-3200
- removed J12: DSP_EN, Connector_PinSocket_2.54mm:PinSocket_1x02_P2.54mm_Vertical
- removed J13: OUT1, XKB_PJ-3200:XKB_PJ-3200
- removed J14: OUT2, XKB_PJ-3200:XKB_PJ-3200
- removed J15: SELFBOOT, Connector_PinHeader_2.54mm:PinHeader_1x03_P2.54mm_Vertical
- removed J16: DSP_PROG, Connector_PinSocket_2.54mm:PinSocket_1x05_P2.54mm_Vertical
- removed J17: DSP_GPIO, Connector_PinHeader_2.54mm:PinHeader_2x07_P2.54mm_Vertical
- removed Q2: BC807, Package_TO_SOT_SMD:SOT-23
- removed R30, R31, R37: 18K, Resistor_SMD:R_0603_1608Metric_Pad0.98x0.95mm_HandSolder
- removed R32, R33: 49.9k, Resistor_SMD:R_0603_1608Metric_Pad0.98x0.95mm_HandSolder
- removed R34, R35, R36: 10k, Resistor_SMD:R_0603_1608Metric_Pad0.98x0.95mm_HandSolder
- removed R38: 470R, Resistor_SMD:R_0603_1608Metric_Pad0.98x0.95mm_HandSolder
- removed R39: 100R, Resistor_SMD:R_0603_1608Metric_Pad0.98x0.95mm_HandSolder
- removed R40, R41, R42, R43: 560R, Resistor_SMD:R_0603_1608Metric_Pad0.98x0.95mm_HandSolder
- removed R44: 10K, Resistor_SMD:R_0603_1608Metric_Pad0.98x0.95mm_HandSolder
- removed R45: 1K, Resistor_SMD:R_0603_1608Metric_Pad0.98x0.95mm_HandSolder
- removed SW1: DSP_RST, TS3425BA:TS3425BA
- removed TP15: V_DSP, TestPoint:TestPoint_THTPad_1.0x1.0mm_Drill0.5mm
- removed TP16: 3.3V, TestPoint:TestPoint_THTPad_1.0x1.0mm_Drill0.5mm
- removed TP17: O1_R, TestPoint:TestPoint_THTPad_1.0x1.0mm_Drill0.5mm
- removed TP18: O1_L, TestPoint:TestPoint_THTPad_1.0x1.0mm_Drill0.5mm
- removed TP19: O2_R, TestPoint:TestPoint_THTPad_1.0x1.0mm_Drill0.5mm
- removed TP20: O2_L, TestPoint:TestPoint_THTPad_1.0x1.0mm_Drill0.5mm
- removed U4: ADAU1701, Package_QFP:LQFP-48_7x7mm_P0.5mm
- removed U5: M24C64-RMN6TP, Package_SO:SOIC-8_3.9x4.9mm_P1.27mm
- removed Y2: XTM32012288JT00351001, Crystal:Crystal_SMD_3225-4Pin_3.2x2.5mm_HandSoldering
Connections:
- D4 pad 2: unconnected-(R28-Pad1) -> Net-(D4-A)
- JP8 pad 1: unconnected-(R27-Pad2) -> Net-(JP8-A)
- R26 pad 2: unconnected-(R26-Pad2) -> Net-(U3-NC)
- R27 pad 2: unconnected-(R27-Pad2) -> Net-(JP8-A)
- R28 pad 1: unconnected-(R28-Pad1) -> Net-(D4-A)
- U3 pad 18: (no net) -> unconnected-(U3-P0.12/I2S_MCLK-Pad18)
- U3 pad 9: unconnected-(R26-Pad2) -> Net-(U3-NC)
Routing:
- net unconnected-(R27-Pad2): track 3.54 -> 0.00 mm
- net Net-(JP8-A): track 0.00 -> 3.54 mm
- net unconnected-(R28-Pad1): track 3.28 -> 0.00 mm
- net Net-(D4-A): track 0.00 -> 3.28 mm
- net unconnected-(R26-Pad2): track 2.80 -> 0.00 mm
- net Net-(U3-NC): track 0.00 -> 2.80 mm
Other:
- board text removed: "SBOOT"
- board text removed: "VDSP"
- board text removed: "WP"
