File: FSC-BT631D-Breakout/FSC-BT631D-Breakout.kicad_sch (KiCad schematic)
At the start: 0 parts

Commit message: folder restructure
Other:
- removed sheet DSP
Changed lines of the file:
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@@
 	(paper "A4")
-	(sheet
-		(at 125.73 63.5)
-		(size 16.51 12.7)
-		(exclude_from_sim no)
-		(in_bom yes)
-		(on_board yes)
-		(dnp no)
-		(fields_autoplaced yes)
-		(stroke
-			(width 0.1524)
-			(type solid)
-		)
-		(fill
-			(color 0 0 0 0.0000)
-		)
-		(property "Sheetname" "DSP"
-			(at 125.73 62.7884 0)
-			(effects
-				(font
-					(size 1.27 1.27)
-				)
-				(justify left bottom)
-			)
-		)
-		(property "Sheetfile" "dsp.kicad_sch"
-			(at 125.73 76.7846 0)
-			(effects
-				(font
-					(size 1.27 1.27)
-				)
-				(justify left top)
-			)
-		)
-		(instances
-			(project "FSC-BT631D-Breakout"
-				(path "/484c4955-80b8-457c-864e-1c65a3218727"
-					(page "6")
-				)
-			)
-		)
-	)
 	(sheet
 		(at 102.87 63.5)
