File: ADAU1701-DSP/ADAU1701-DSP.kicad_pcb (KiCad board)
At the start: 2 copper layers, 67 parts, among them J11 DSP IN, J12 VIN, J13 OUT1, J14 OUT2, J15 SELFBOOT, J16 DSP_PROG, J17 DSP_GPIO, Q2 BC807, SW1 DSP_RST, U4 ADAU1701, U5 M24C64-RMN6TP, Y2 XTM32012288JT00351001

Commit message: dsp routing finished
Parts:
- removed C34: 3.3nF, Capacitor_SMD:C_0603_1608Metric_Pad1.08x0.95mm_HandSolder
- removed C35: 47nF, Capacitor_SMD:C_0603_1608Metric_Pad1.08x0.95mm_HandSolder
- removed C36, C37: 22pF, Capacitor_SMD:C_0603_1608Metric_Pad1.08x0.95mm_HandSolder
- removed C38, C41, C44, C45: 5.6nF, Capacitor_SMD:C_0603_1608Metric_Pad1.08x0.95mm_HandSolder
- removed C39, C40, C42, C43: 47uF, Capacitor_SMD:C_0603_1608Metric_Pad1.08x0.95mm_HandSolder
- removed C46, C47, C48, C50, C51, C52, C55: 100nF, Capacitor_SMD:C_0603_1608Metric_Pad1.08x0.95mm_HandSolder
- removed C49: 100uF, Capacitor_SMD:C_0603_1608Metric_Pad1.08x0.95mm_HandSolder
- removed C53, C54: 10uF, Capacitor_SMD:C_0603_1608Metric_Pad1.08x0.95mm_HandSolder
- removed J11: DSP IN, XKB_PJ-3200:XKB_PJ-3200
- removed J12: VIN, Connector_PinSocket_2.54mm:PinSocket_1x02_P2.54mm_Vertical
- removed J13: OUT1, XKB_PJ-3200:XKB_PJ-3200
- removed J14: OUT2, XKB_PJ-3200:XKB_PJ-3200
- removed J15: SELFBOOT, Connector_PinHeader_2.54mm:PinHeader_1x03_P2.54mm_Vertical
- removed J16: DSP_PROG, Connector_PinSocket_2.54mm:PinSocket_1x05_P2.54mm_Vertical
- removed J17: DSP_GPIO, Connector_PinHeader_2.54mm:PinHeader_2x07_P2.54mm_Vertical
- removed Q2: BC807, Package_TO_SOT_SMD:SOT-23
- removed R30, R31, R37: 18K, Resistor_SMD:R_0603_1608Metric_Pad0.98x0.95mm_HandSolder
- removed R32, R33: 49.9k, Resistor_SMD:R_0603_1608Metric_Pad0.98x0.95mm_HandSolder
- removed R34, R35, R36: 10k, Resistor_SMD:R_0603_1608Metric_Pad0.98x0.95mm_HandSolder
- removed R38: 470R, Resistor_SMD:R_0603_1608Metric_Pad0.98x0.95mm_HandSolder
- removed R39: 100R, Resistor_SMD:R_0603_1608Metric_Pad0.98x0.95mm_HandSolder
- removed R40, R41, R42, R43: 560R, Resistor_SMD:R_0603_1608Metric_Pad0.98x0.95mm_HandSolder
- removed R44: 10K, Resistor_SMD:R_0603_1608Metric_Pad0.98x0.95mm_HandSolder
- removed R45: 1K, Resistor_SMD:R_0603_1608Metric_Pad0.98x0.95mm_HandSolder
- removed TP15: GND, TestPoint:TestPoint_THTPad_1.0x1.0mm_Drill0.5mm
- removed TP16: 3.3V, TestPoint:TestPoint_THTPad_1.0x1.0mm_Drill0.5mm
- removed TP17: O1_R, TestPoint:TestPoint_THTPad_1.0x1.0mm_Drill0.5mm
- removed TP18: O1_L, TestPoint:TestPoint_THTPad_1.0x1.0mm_Drill0.5mm
- removed TP19: O2_R, TestPoint:TestPoint_THTPad_1.0x1.0mm_Drill0.5mm
- removed TP20: O2_L, TestPoint:TestPoint_THTPad_1.0x1.0mm_Drill0.5mm
- removed U4: ADAU1701, Package_QFP:LQFP-48_7x7mm_P0.5mm
- removed U5: M24C64-RMN6TP, Package_SO:SOIC-8_3.9x4.9mm_P1.27mm
- removed Y2: XTM32012288JT00351001, Crystal:Crystal_SMD_3225-4Pin_3.2x2.5mm_HandSoldering
- added C1: 47uF, Capacitor_SMD:C_0603_1608Metric_Pad1.08x0.95mm_HandSolder, F.Cu at (177.8, 130.4)
- added C10: 10uF, Capacitor_SMD:C_0603_1608Metric_Pad1.08x0.95mm_HandSolder, F.Cu at (185.4, 120.7)
- added C11: 100nF, Capacitor_SMD:C_0603_1608Metric_Pad1.08x0.95mm_HandSolder, F.Cu at (167.6, 113.0)
- added C12: 22pF, Capacitor_SMD:C_0603_1608Metric_Pad1.08x0.95mm_HandSolder, F.Cu at (190.5, 120.0)
- added C13: 100nF, Capacitor_SMD:C_0603_1608Metric_Pad1.08x0.95mm_HandSolder, F.Cu at (167.6, 116.8)
- added C14: 47uF, Capacitor_SMD:C_0603_1608Metric_Pad1.08x0.95mm_HandSolder, F.Cu at (165.1, 116.8)
- added C15: 100nF, Capacitor_SMD:C_0603_1608Metric_Pad1.08x0.95mm_HandSolder, F.Cu at (182.9, 120.7)
- added C16: 100nF, Capacitor_SMD:C_0603_1608Metric_Pad1.08x0.95mm_HandSolder, F.Cu at (170.2, 113.0)
- added C17: 22pF, Capacitor_SMD:C_0603_1608Metric_Pad1.08x0.95mm_HandSolder, F.Cu at (190.5, 111.1)
- added C18: 100nF, Capacitor_SMD:C_0603_1608Metric_Pad1.08x0.95mm_HandSolder, F.Cu at (172.7, 113.0)
- added C19: 100nF, Capacitor_SMD:C_0603_1608Metric_Pad1.08x0.95mm_HandSolder, F.Cu at (167.6, 120.7)
- added C2: 100nF, Capacitor_SMD:C_0603_1608Metric_Pad1.08x0.95mm_HandSolder, F.Cu at (165.1, 124.5)
- added C20: 10uF, Capacitor_SMD:C_0603_1608Metric_Pad1.08x0.95mm_HandSolder, F.Cu at (165.1, 120.7)
- added C21: 100nF, Capacitor_SMD:C_0603_1608Metric_Pad1.08x0.95mm_HandSolder, F.Cu at (188.0, 130.4)
- added C22: 100nF, Capacitor_SMD:C_0603_1608Metric_Pad1.08x0.95mm_HandSolder, F.Cu at (185.4, 130.4)
- added C3: 10uF, Capacitor_SMD:C_0603_1608Metric_Pad1.08x0.95mm_HandSolder, F.Cu at (167.6, 124.5)
- added C4: 3.3nF, Capacitor_SMD:C_0603_1608Metric_Pad1.08x0.95mm_HandSolder, F.Cu at (175.3, 113.0)
- added C5: 10uF, Capacitor_SMD:C_0603_1608Metric_Pad1.08x0.95mm_HandSolder, F.Cu at (165.1, 113.0)
- added C6: 47nF, Capacitor_SMD:C_0603_1608Metric_Pad1.08x0.95mm_HandSolder, F.Cu at (177.8, 113.0)
- added C7: 47uF, Capacitor_SMD:C_0603_1608Metric_Pad1.08x0.95mm_HandSolder, F.Cu at (165.1, 130.4)
- added C8: 100pF, Capacitor_SMD:C_0603_1608Metric_Pad1.08x0.95mm_HandSolder, F.Cu at (162.6, 130.4)
- added C9: 100pF, Capacitor_SMD:C_0603_1608Metric_Pad1.08x0.95mm_HandSolder, F.Cu at (175.3, 130.4)
- added J2: VIN, Connector_PinSocket_2.54mm:PinSocket_1x02_P2.54mm_Vertical, F.Cu at (198.1, 104.1)
- added J3: SELFBOOT, Connector_PinHeader_2.54mm:PinHeader_1x03_P2.54mm_Vertical, F.Cu at (154.9, 134.6)
- added J4: IO1, Connector_PinSocket_2.54mm:PinSocket_1x15_P2.54mm_Vertical, F.Cu at (190.5, 104.1)
- added J5: IO2, Connector_PinSocket_2.54mm:PinSocket_1x15_P2.54mm_Vertical, F.Cu at (200.7, 134.9)
- added Q1: BC807, Package_TO_SOT_SMD:SOT-23, F.Cu at (184.2, 125.3)
- added R1: 18K, Resistor_SMD:R_0603_1608Metric_Pad0.98x0.95mm_HandSolder, F.Cu at (180.3, 130.4)
- added R10: 560R, Resistor_SMD:R_0603_1608Metric_Pad0.98x0.95mm_HandSolder, F.Cu at (160.0, 116.8)
- added R11: 10K, Resistor_SMD:R_0603_1608Metric_Pad0.98x0.95mm_HandSolder, F.Cu at (162.6, 124.5)
- added R12: 560R, Resistor_SMD:R_0603_1608Metric_Pad0.98x0.95mm_HandSolder, F.Cu at (157.5, 116.8)
- added R13: 560R, Resistor_SMD:R_0603_1608Metric_Pad0.98x0.95mm_HandSolder, F.Cu at (162.6, 116.8)
- added R14: 10k, Resistor_SMD:R_0603_1608Metric_Pad0.98x0.95mm_HandSolder, F.Cu at (194.3, 130.4)
- added R15: 10k, Resistor_SMD:R_0603_1608Metric_Pad0.98x0.95mm_HandSolder, F.Cu at (196.8, 130.4)
- added R16: 10k, Resistor_SMD:R_0603_1608Metric_Pad0.98x0.95mm_HandSolder, F.Cu at (199.4, 130.4)
- added R2: 470R, Resistor_SMD:R_0603_1608Metric_Pad0.98x0.95mm_HandSolder, F.Cu at (180.3, 113.0)
- added R3: 18K, Resistor_SMD:R_0603_1608Metric_Pad0.98x0.95mm_HandSolder, F.Cu at (167.6, 130.4)
- added R4: 49.9k, Resistor_SMD:R_0603_1608Metric_Pad0.98x0.95mm_HandSolder, F.Cu at (160.0, 130.4)
- added R5: 49.9k, Resistor_SMD:R_0603_1608Metric_Pad0.98x0.95mm_HandSolder, F.Cu at (172.7, 130.4)
- added R6: 100R, Resistor_SMD:R_0603_1608Metric_Pad0.98x0.95mm_HandSolder, F.Cu at (185.4, 115.6)
- added R7: 1K, Resistor_SMD:R_0603_1608Metric_Pad0.98x0.95mm_HandSolder, F.Cu at (188.0, 125.3)
- added R8: 18K, Resistor_SMD:R_0603_1608Metric_Pad0.98x0.95mm_HandSolder, F.Cu at (170.2, 130.4)
- added R9: 560R, Resistor_SMD:R_0603_1608Metric_Pad0.98x0.95mm_HandSolder, F.Cu at (154.9, 116.8)
- added TP1: 3.3V, TestPoint:TestPoint_THTPad_1.0x1.0mm_Drill0.5mm, F.Cu at (198.1, 109.2)
- added TP2: GND, TestPoint:TestPoint_THTPad_1.0x1.0mm_Drill0.5mm, F.Cu at (200.7, 109.2)
- added TP3: O1_R, TestPoint:TestPoint_THTPad_1.0x1.0mm_Drill0.5mm, F.Cu at (157.5, 109.2)
- added TP4: O2_R, TestPoint:TestPoint_THTPad_1.0x1.0mm_Drill0.5mm, F.Cu at (162.6, 109.2)
- added TP5: O1_L, TestPoint:TestPoint_THTPad_1.0x1.0mm_Drill0.5mm, F.Cu at (160.0, 109.2)
- added TP6: O2_L, TestPoint:TestPoint_THTPad_1.0x1.0mm_Drill0.5mm, F.Cu at (165.1, 109.2)
- added U1: ADAU1701, Package_QFP:LQFP-48_7x7mm_P0.5mm, F.Cu at (175.3, 121.2)
- added U2: M24C64-RMN6TP, Package_SO:SOIC-8_3.9x4.9mm_P1.27mm, F.Cu at (196.8, 122.8)
- added Y1: XTM32012288JT00351001, Crystal:Crystal_SMD_3225-4Pin_3.2x2.5mm_HandSoldering, F.Cu at (190.5, 115.6)
- C23: value 100pF -> 100uF
- C24: value 100pF -> 47uF
- C26, C31: value 47uF -> 5.6nF
- C27, C30: value 100nF -> 5.6nF
- C28: value 100nF -> 47uF
- C29: value 10uF -> 47uF
- C33: value 10uF -> 100nF
- moved C23 60.4 mm to (182.9, 130.4)
- moved C33 50.0 mm to (201.9, 122.8), turned to 90 degrees
- moved C32 45.7 mm to (154.9, 124.5), turned to 90 degrees
- moved C24 44.5 mm to (154.9, 120.7)
- moved C28 39.0 mm to (157.5, 120.7)
- moved C30 37.8 mm to (157.5, 113.0), turned to 90 degrees
- moved C29 37.6 mm to (162.6, 120.7)
- moved C27 33.6 mm to (160.0, 113.0), turned to 90 degrees
- moved C31 33.4 mm to (162.6, 113.0), turned to 90 degrees
- moved C25 32.6 mm to (160.0, 120.7), turned to -90 degrees
- moved SW1 29.9 mm to (158.8, 125.7)
- moved C26 21.7 mm to (154.9, 113.0), turned to 90 degrees
Connections:
- C23 pad 1: GND -> /DVDD
- C23 pad 2: /DSP_IN_LEFT -> GND
- C24 pad 1: GND -> Net-(C24-Pad1)
- C24 pad 2: /DSP_IN_RIGHT -> /VOUT0
- C25 pad 2: /DSP_IN_LEFT -> /VOUT2
- C26 pad 1: Net-(C26-Pad1) -> /OUT1_R
- C26 pad 2: /DSP_IN_RIGHT -> GND
- C27 pad 1: +3.3V -> /OUT2_R
- C28 pad 1: GND -> Net-(C28-Pad1)
- C28 pad 2: /FILTA -> /VOUT1
- C29 pad 1: GND -> Net-(C29-Pad1)
- C29 pad 2: /FILTA -> /VOUT3
- C30 pad 1: GND -> /OUT1_L
- C30 pad 2: /CM -> GND
- C31 pad 1: GND -> /OUT2_L
- C31 pad 2: /CM -> GND
- C32 pad 2: /FILTD -> /DSP_RST
- C33 pad 1: GND -> +3.3V
- C33 pad 2: /FILTD -> GND
Routing:
- net /DSP_SDA: track 3.23 -> 42.6 mm, vias 0 -> 2
- net +3.3V: track 105.2 -> 143.7 mm, vias 7 -> 0
- net /DSP_SCL: track 4.01 -> 41.5 mm, vias 0 -> 2
- net /DSP_WP: track 5.88 -> 36.9 mm, vias 0 -> 1
- net /VOUT2: track 42.2 -> 12.2 mm, vias 2 -> 0
- net /VOUT3: track 39.3 -> 9.34 mm, vias 2 -> 0
- net /DSP_RST: track 18.8 -> 48.4 mm, vias 0 -> 2
- net /MP11: track 0.00 -> 28.9 mm, vias 0 -> 1
- net /SBOOT: track 0.00 -> 25.1 mm, vias 0 -> 2
- net /VOUT0: track 42.2 -> 17.4 mm
- net /VOUT1: track 38.6 -> 15.0 mm
- net /MP10: track 0.00 -> 20.9 mm, vias 0 -> 1
- net /DSP_IN_LEFT: track 18.2 -> 0.00 mm
- net /DSP_IN_RIGHT: track 17.8 -> 0.00 mm
- net GND: track 0.00 -> 16.9 mm, vias 0 -> 303
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- added copper zone on B.Cu, net GND
- added copper zone on F.Cu, net GND
Other:
- board outline added: 53.3 x 35.6 mm
- board text added: "3.3v"
- board text added: "INL"
- board text added: "INR"
- board text added: "O1"
- board text added: "O2"
- board text added: "O3"
- board text added: "O4"
- board text added: "RST"
- board text removed: "VDSP"
