File: ADAU1701-DSP/ADAU1701-DSP.kicad_sch (KiCad schematic)
At the start: 67 parts, among them J11 DSP IN, J12 VIN, J13 OUT1, J14 OUT2, J15 SELFBOOT, J16 DSP_PROG, J17 DSP_GPIO, Q2 BC807, SW1 DSP_RST, U4 ADAU1701, U5 M24C64-RMN6TP, Y2 XTM32012288JT00351001

Commit message: dsp routing finished
Parts:
- removed J11: DSP IN, XKB_PJ-3200:XKB_PJ-3200, symbol Connector_Audio:AudioJack2_Ground
- removed J13: OUT1, XKB_PJ-3200:XKB_PJ-3200, symbol Connector_Audio:AudioJack2_Ground
- removed J14: OUT2, XKB_PJ-3200:XKB_PJ-3200, symbol Connector_Audio:AudioJack2_Ground
- removed J16: DSP_PROG, Connector_PinSocket_2.54mm:PinSocket_1x05_P2.54mm_Vertical, symbol Connector_Generic:Conn_01x05
- removed J17: DSP_GPIO, Connector_PinHeader_2.54mm:PinHeader_2x07_P2.54mm_Vertical, symbol Connector_Generic:Conn_02x07_Odd_Even
- added J4: IO1, Connector_PinSocket_2.54mm:PinSocket_1x15_P2.54mm_Vertical, symbol Connector_Generic:Conn_01x15
- added J5: IO2, Connector_PinSocket_2.54mm:PinSocket_1x15_P2.54mm_Vertical, symbol Connector_Generic:Conn_01x15
- renumbered C26 to C1, C54 to C10, C52 to C11, C36 to C12, C30 to C13, C31 to C14, C55 to C15, C51 to C16, C37 to C17, C50 to C18, C32 to C19, C28 to C2, C33 to C20, C47 to C21, C48 to C22, C49 to C23, C39 to C24, C42 to C25, C38 to C26, C44 to C27, C40 to C28, C43 to C29, C29 to C3, C41 to C30, C45 to C31, C46 to C32, C27 to C33, C34 to C4, C53 to C5, C35 to C6, C25 to C7, C23 to C8, C24 to C9, J12 to J2, J15 to J3, Q2 to Q1, R31 to R1, R42 to R10, R44 to R11, R41 to R12, R43 to R13, R34 to R14, R35 to R15, R36 to R16, R38 to R2, R30 to R3, R32 to R4, R33 to R5, R39 to R6, R45 to R7, R37 to R8, R40 to R9, TP16 to TP1, TP15 to TP2, TP17 to TP3, TP19 to TP4, TP18 to TP5, TP20 to TP6, U4 to U1, U5 to U2, Y2 to Y1
Connections:
- net V_DSP is gone; now on net +3.3V: J3.1 (Pin_1)
- net +3.3V: now also J4.1 (Pin_1)
- net DSP_RST: now also J4.4 (Pin_4)
- net DSP_SCL: now also J4.3 (Pin_3)
- net DSP_SDA: now also J4.2 (Pin_2)
- net DSP_WP: now also J5.1 (Pin_1)
- net GND: now also J4.10 (Pin_10), J4.15 (Pin_15), J4.5 (Pin_5), J5.12 (Pin_12), J5.14 (Pin_14), J5.15 (Pin_15), J5.2 (Pin_2)
- net MP0: now also J5.7 (Pin_7)
- net MP1: now also J5.8 (Pin_8)
- net MP10: now also J5.4 (Pin_4)
- net MP11: now also J5.3 (Pin_3)
- net MP2: now also J4.9 (Pin_9)
- net MP3: now also J4.8 (Pin_8)
- net MP4: now also J5.10 (Pin_10)
- net MP5: now also J5.9 (Pin_9)
- net MP6: now also J5.5 (Pin_5)
- net MP7: now also J5.6 (Pin_6)
- net MP8: now also J4.7 (Pin_7)
- net MP9: now also J4.6 (Pin_6)
- net DSP_IN_LEFT renamed DSP_IN_L
- net DSP_IN_L: now also J5.13 (Pin_13)
- net DSP_IN_RIGHT renamed DSP_IN_R
- net DSP_IN_R: now also J5.11 (Pin_11)
- net OUT1_LEFT renamed OUT1_L
- net OUT1_L: now also J4.13 (Pin_13)
- net OUT1_RIGHT renamed OUT1_R
- net OUT1_R: now also J4.14 (Pin_14)
- net OUT2_LEFT renamed OUT2_L
- net OUT2_L: now also J4.11 (Pin_11)
- net OUT2_RIGHT renamed OUT2_R
- net OUT2_R: now also J4.12 (Pin_12)
